Commit message: Made tweaks to urdf

File: src/robodog_gazebo/urdf/robodog_skeleton.urdf (robot description, URDF)
Before this commit: robot robodog_skeleton, 21 links, 20 joints
Joints:
- joint front_left_base_hip_joint: axis 0 0 1 -> 1 0 0
- joint front_left_hip_1_hip_2_joint: axis (none) -> 0.0 0.0 1.0; limit (none) -> lower=-3.1415926 upper=3.1415926 effort=1000 velocity=1.0; origin xyz=${hip_1_half_length} 0.0 0.0 rpy=0.0 0.0 0.0 -> xyz=${2 * hip_1_half_width} 0.0 0.0 rpy=0.0 0.0 0.0; type fixed -> revolute
- joint front_left_hip_tibia_joint: axis 0.0 0.0 1.0 -> (none); limit lower=-3.1415926 upper=3.1415926 effort=1000 velocity=1.0 -> (none); type revolute -> fixed
- joint front_right_base_hip_joint: axis 0 0 1 -> 1 0 0
- joint front_right_hip_1_hip_2_joint: axis (none) -> 0.0 0.0 1.0; limit (none) -> lower=-3.1415926 upper=3.1415926 effort=1000 velocity=1.0; origin xyz=${hip_1_half_length} 0.0 0.0 rpy=0.0 0.0 0.0 -> xyz=${2 * hip_1_half_width} 0.0 0.0 rpy=0.0 0.0 0.0; type fixed -> revolute
- joint front_right_hip_tibia_joint: axis 0.0 0.0 1.0 -> (none); limit lower=-3.1415926 upper=3.1415926 effort=1000 velocity=1.0 -> (none); type revolute -> fixed
- joint rear_left_base_hip_joint: axis 0 0 1 -> 1 0 0
- joint rear_left_hip_1_hip_2_joint: axis (none) -> 0.0 0.0 1.0; limit (none) -> lower=-3.1415926 upper=3.1415926 effort=1000 velocity=1.0; origin xyz=${hip_1_half_length} 0.0 0.0 rpy=0.0 0.0 0.0 -> xyz=${2 * hip_1_half_width} 0.0 0.0 rpy=0.0 0.0 0.0; type fixed -> revolute
- joint rear_left_hip_tibia_joint: axis 0.0 0.0 1.0 -> (none); limit lower=-3.1415926 upper=3.1415926 effort=1000 velocity=1.0 -> (none); type revolute -> fixed
- joint rear_right_base_hip_joint: axis 0 0 1 -> 1 0 0
- joint rear_right_hip_1_hip_2_joint: axis (none) -> 0.0 0.0 1.0; limit (none) -> lower=-3.1415926 upper=3.1415926 effort=1000 velocity=1.0; origin xyz=${hip_1_half_length} 0.0 0.0 rpy=0.0 0.0 0.0 -> xyz=${2 * hip_1_half_width} 0.0 0.0 rpy=0.0 0.0 0.0; type fixed -> revolute
- joint rear_right_hip_tibia_joint: axis 0.0 0.0 1.0 -> (none); limit lower=-3.1415926 upper=3.1415926 effort=1000 velocity=1.0 -> (none); type revolute -> fixed

Commit message: Updated urdf shoulders to overlap properly

File: src/robodog_gazebo/urdf/robodog_skeleton.urdf (robot description, URDF)
Before this commit: robot robodog_skeleton, 21 links, 20 joints
Joints:
- joint front_left_hip_1_hip_2_joint: origin xyz=${2 * hip_1_half_width} 0.0 0.0 rpy=0.0 0.0 0.0 -> xyz=${hip_1_width-hip_2_width/2} -0.0073 0.0 rpy=0.0 0.0 0.0
- joint front_right_hip_1_hip_2_joint: origin xyz=${2 * hip_1_half_width} 0.0 0.0 rpy=0.0 0.0 0.0 -> xyz=${hip_1_width-hip_2_width/2} -0.0073 0.0 rpy=0.0 0.0 0.0
- joint rear_left_hip_1_hip_2_joint: origin xyz=${2 * hip_1_half_width} 0.0 0.0 rpy=0.0 0.0 0.0 -> xyz=${hip_1_width-hip_2_width/2} -0.0073 0.0 rpy=0.0 0.0 0.0
- joint rear_right_hip_1_hip_2_joint: origin xyz=${2 * hip_1_half_width} 0.0 0.0 rpy=0.0 0.0 0.0 -> xyz=${hip_1_width-hip_2_width/2} -0.0073 0.0 rpy=0.0 0.0 0.0
