Commit message: Updated controls to work on imported model

File: src/try_again_i_guess/urdf/try_again_i_guess.urdf (robot description, URDF)
Before this commit: robot try_again_i_guess, 17 links, 16 joints
Joints:
- joint joint_BL1: limit (none) -> lower=-3.1415926 upper=3.1415926 effort=1000 velocity=1.0; type continuous -> revolute
- joint joint_BL2: limit (none) -> lower=-3.1415926 upper=3.1415926 effort=1000 velocity=1.0; type continuous -> revolute
- joint joint_BL3: limit (none) -> lower=-3.1415926 upper=3.1415926 effort=1000 velocity=1.0; type continuous -> revolute
- joint joint_BR1: limit (none) -> lower=-3.1415926 upper=3.1415926 effort=1000 velocity=1.0; type continuous -> revolute
- joint joint_BR2: limit (none) -> lower=-3.1415926 upper=3.1415926 effort=1000 velocity=1.0; type continuous -> revolute
- joint joint_BR3: limit (none) -> lower=-3.1415926 upper=3.1415926 effort=1000 velocity=1.0; type continuous -> revolute
- joint joint_FL1: limit (none) -> lower=-3.1415926 upper=3.1415926 effort=1000 velocity=1.0; type continuous -> revolute
- joint joint_FL2: limit (none) -> lower=-3.1415926 upper=3.1415926 effort=1000 velocity=1.0; type continuous -> revolute
- joint joint_FL3: limit (none) -> lower=-3.1415926 upper=3.1415926 effort=1000 velocity=1.0; type continuous -> revolute
- joint joint_FR1: limit (none) -> lower=-3.1415926 upper=3.1415926 effort=1000 velocity=1.0; type continuous -> revolute
- joint joint_FR2: limit (none) -> lower=-3.1415926 upper=3.1415926 effort=1000 velocity=1.0; type continuous -> revolute
- joint joint_FR3: limit (none) -> lower=-3.1415926 upper=3.1415926 effort=1000 velocity=1.0; type continuous -> revolute
