Commit message: Fixed Odometry (Localization)

File: src/urdf_color/urdf/urdf_color.urdf.xacro (robot description, xacro)
@@ -8,4 +8,11 @@
     <origin xyz="0 0 0" rpy="0 0 0" />
   </xacro:zed_camera>
+  <link name="base_footprint"/>
+  <joint name="base_joint" type="fixed">
+    <parent link="base_footprint"/>
+    <child link="base_link"/>
+    <!-- Center the robot, ground it, and rotate -90 deg so X is forward -->
+    <origin xyz="0.8858 0.8375 -0.7894" rpy="0 0 -1.5708" />
+  </joint>
   <link name="base_link">
     <inertial>
@@ -350,5 +357,5 @@
       <origin xyz="-0.00313707084207038 -0.113584540455344 -0.042496272818598" rpy="0 0 0" />
       <mass value="0.228830429344516" />
-      <inertia ixx="0.000231457353091744" ixy="5.80698239952246E-09" ixz="-5.80606638398738E-09" iyy="0.000106373346469612" iyz="-1.13763375269897E-05" izz="0.000209650486510219" />
+      <inertia ixx="0.000231457353091744" ixy="5.80698239952246E-09" ixz="-5.80606638398738E-09" iyy="0.000106373346469612" iyz="-1.137633375269897E-05" izz="0.000209650486510219" />
     </inertial>
     <visual>
@@ -730,5 +737,5 @@
     <plugin filename="gz-sim-odometry-publisher-system" name="gz::sim::systems::OdometryPublisher">
       <odom_frame>odom</odom_frame>
-      <robot_base_frame>base_link</robot_base_frame>
+      <robot_base_frame>base_footprint</robot_base_frame>
       <odom_topic>zed/zed_node/odom</odom_topic>
       <tf_topic>zed/zed_node/tf</tf_topic>

Commit message: Virtual Commands

File: src/urdf_color/urdf/urdf_color.urdf.xacro (robot description, xacro)
@@ -8,5 +8,11 @@
     <origin xyz="0 0 0" rpy="0 0 0" />
   </xacro:zed_camera>
-  <link name="base_footprint"/>
+  <link name="base_footprint">
+    <inertial>
+      <mass value="0.0001"/>
+      <origin xyz="0 0 0"/>
+      <inertia ixx="0.0001" ixy="0.0" ixz="0.0" iyy="0.0001" iyz="0.0" izz="0.0001"/>
+    </inertial>
+  </link>
   <joint name="base_joint" type="fixed">
     <parent link="base_footprint"/>
